File: corne-light/pcb/corne-light.sch (KiCad schematic (older format))
At the start: 92 parts, among them J1 MJ-4PP-9, J2 OLED, J6 MJ-4PP-9, J7 OLED, SW1 SW_PUSH, SW10 SW_PUSH, SW11 SW_PUSH, SW12 SW_PUSH, SW13 SW_PUSH, SW14 SW_PUSH, SW15 SW_PUSH, SW16 SW_PUSH, SW17 SW_PUSH, SW18 SW_PUSH, SW19 SW_PUSH, SW2 SW_PUSH, SW20 SW_PUSH, SW21 SW_PUSH, SW22 SW_PUSH, SW23 SW_PUSH, SW24 SW_PUSH, SW25 SW_PUSH, SW26 SW_PUSH, SW27 SW_PUSH, SW28 SW_PUSH, SW29 SW_PUSH, SW3 SW_PUSH, SW30 SW_PUSH, SW31 SW_PUSH, SW32 SW_PUSH, SW33 SW_PUSH, SW34 SW_PUSH, SW35 SW_PUSH, SW36 SW_PUSH, SW37 SW_PUSH, SW38 SW_PUSH, SW39 SW_PUSH, SW4 SW_PUSH, SW40 SW_PUSH, SW41 SW_PUSH, SW42 SW_PUSH, SW5 SW_PUSH, SW6 SW_PUSH, SW7 SW_PUSH, SW8 SW_PUSH, SW9 SW_PUSH, U1 ProMicro, U2 ProMicro

Commit message: Change to CCDs
Parts:
- removed D1, D10, D11, D12, D13, D14, D15, D16, D17, D18, D19, D2, D20, D21, D22, D23, D24, D25, D26, D27, D28, D29, D3, D30, D31, D32, D33, D34, D35, D36, D37, D38, D39, D4, D40, D41, D42, D5, D6, D7, D8, D9: D, kbd:D3_TH, symbol Device:D
- added D1, D10, D11, D12, D13, D14, D15, D16, D17, D18, D19, D2, D20, D21, D22, D3, D4, D5, D6, D7, D8, D9: BAV70, Custom_Footprints:SOT-23_Annotated, symbol Diode:BAV70
- SW1, SW10, SW11, SW12, SW13, SW14, SW15, SW16, SW17, SW18, SW19, SW2, SW20, SW22, SW23, SW24, SW25, SW26, SW27, SW28, SW29, SW3, SW30, SW31, SW32, SW33, SW34, SW35, SW36, SW37, SW38, SW39, SW4, SW40, SW41, SW5, SW6, SW7, SW8, SW9: footprint kbd:CherryMX_ChocV2_1u -> MX_Only:MXOnly-1U-NoLED
- SW21, SW42: footprint kbd:CherryMX_ChocV2_1.5u -> MX_Only:MXOnly-1.5U-NoLED
Connections:
- wire segments 112 -> 92
- no-connect marks 15 -> 16
Other:
- moved on the sheet: J1, J2, J6, J7, RSW1, RSW2, SW1, SW10, SW11, SW12, SW13, SW14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

Commit message: Place CCDs
Connections:
- net at SW19.2: now also D10.1 (A); no longer D10.2 (A)
- net at SW23.2: now also D12.1 (A); no longer D12.2 (A)
- net at SW24.2: now also D13.2 (A); no longer D13.1 (A)
- net at SW25.2: now also D13.1 (A); no longer D13.2 (A)
- net at SW26.2: now also D14.2 (A); no longer D14.1 (A)
- net at SW27.2: now also D14.1 (A); no longer D14.2 (A)
- net at SW22.2: now also D12.2 (A); no longer D12.1 (A)
- net at SW29.2: now also D15.1 (A); no longer D15.2 (A)
- net at SW30.2: now also D16.2 (A); no longer D16.1 (A)
- net at SW31.2: now also D16.1 (A); no longer D16.2 (A)
- net at SW32.2: now also D17.2 (A); no longer D17.1 (A)
- net at SW33.2: now also D17.1 (A); no longer D17.2 (A)
- net at SW28.2: now also D15.2 (A); no longer D15.1 (A)
- net at SW35.2: now also D18.1 (A); no longer D18.2 (A)
- net at SW36.2: now also D19.2 (A); no longer D19.1 (A)
- net at SW37.2: now also D19.1 (A); no longer D19.2 (A)
- net at SW38.2: now also D20.2 (A); no longer D20.1 (A)
- net at SW39.2: now also D20.1 (A); no longer D20.2 (A)
- net at SW34.2: now also D18.2 (A); no longer D18.1 (A)
- net at SW41.2: now also D22.2 (A); no longer D22.1 (A)
- net at SW42.2: now also D22.1 (A); no longer D22.2 (A)
Changed lines of the file:
@@
 F 3 "https://assets.nexperia.com/documents/data-sheet/BAV70_SER.pdf" H 3900 2725 50  0001 C CNN
 	1    3900 2725
-	1    0    0    -1
+	-1   0    0    -1
 $EndComp
 Wire Wire Line
@@
 F 3 "https://assets.nexperia.com/documents/data-sheet/BAV70_SER.pdf" H 1850 4525 50  0001 C CNN
 	1    1850 4525
-	1    0    0    -1
+	-1   0    0    -1
 $EndComp
 $Comp
@@
 F 3 "https://assets.nexperia.com/documents/data-sheet/BAV70_SER.pdf" H 1850 5025 50  0001 C CNN
 	1    1850 5025
-	1    0    0    -1
+	-1   0    0    -1
 $EndComp
 $Comp
@@
 F 3 "https://assets.nexperia.com/documents/data-sheet/BAV70_SER.pdf" H 1850 5525 50  0001 C CNN
 	1    1850 5525
-	1    0    0    -1
+	-1   0    0    -1
 $EndComp
 $Comp
@@
 F 3 "https://assets.nexperia.com/documents/data-sheet/BAV70_SER.pdf" H 3900 4525 50  0001 C CNN
 	1    3900 4525
-	1    0    0    -1
+	-1   0    0    -1
 $EndComp
 $Comp
@@
 F 3 "https://assets.nexperia.com/documents/data-sheet/BAV70_SER.pdf" H 3900 5025 50  0001 C CNN
 	1    3900 5025
-	1    0    0    -1
+	-1   0    0    -1
 $EndComp
 $Comp
@@
 F 3 "https://assets.nexperia.com/documents/data-sheet/BAV70_SER.pdf" H 3900 5525 50  0001 C CNN
 	1    3900 5525
-	1    0    0    -1
+	-1   0    0    -1
 $EndComp
 $Comp
@@
 F 3 "https://assets.nexperia.com/documents/data-sheet/BAV70_SER.pdf" H 5950 4525 50  0001 C CNN
 	1    5950 4525
-	1    0    0    -1
+	-1   0    0    -1
 $EndComp
 $Comp
@@
 F 3 "https://assets.nexperia.com/documents/data-sheet/BAV70_SER.pdf" H 5950 5025 50  0001 C CNN
 	1    5950 5025
-	1    0    0    -1
+	-1   0    0    -1
 $EndComp
 $Comp
@@
 F 3 "https://assets.nexperia.com/documents/data-sheet/BAV70_SER.pdf" H 5950 5525 50  0001 C CNN
 	1    5950 5525
-	1    0    0    -1
+	-1   0    0    -1
 $EndComp
 $Comp
@@
 F 3 "https://assets.nexperia.com/documents/data-sheet/BAV70_SER.pdf" H 5950 6025 50  0001 C CNN
 	1    5950 6025
-	1    0    0    -1
-$EndComp
-Wire Wire Line
+	-1   0    0    -1
+$EndComp
+Wire Wire Line

Commit message: Route mcu
Connections:
- net col4_r: now also SW41.2; no longer SW41.1
- net col5: now also SW21.2; no longer SW21.1
- net at D11.2 (A): now also SW21.1; no longer SW21.2
- net at D22.2 (A): now also SW41.1; no longer SW41.2
Changed lines of the file:
@@
 F 3 "" H 6550 2725 50  0000 C CNN
 	1    6550 2725
-	-1   0    0    -1
+	1    0    0    -1
 $EndComp
 $Comp
@@
 F 3 "" H 5350 6025 50  0000 C CNN
 	1    5350 6025
-	1    0    0    -1
-$EndComp
-$Comp
+	-1   0    0    -1
+$EndComp
+$Comp
