File: corne-light/pcb/corne-light.kicad_pcb (KiCad board)
At the start: 2 copper layers, 275.5 x 105.6 mm, 122 parts, among them J1 MJ-4PP-9, J2 OLED, J5 Breakaway_Tabs, J6 MJ-4PP-9, J7 OLED, SW1 SW_PUSH, SW10 SW_PUSH, SW11 SW_PUSH, SW12 SW_PUSH, SW13 SW_PUSH, SW14 SW_PUSH, SW15 SW_PUSH, SW16 SW_PUSH, SW17 SW_PUSH, SW18 SW_PUSH, SW19 SW_PUSH, SW2 SW_PUSH, SW20 SW_PUSH, SW21 SW_PUSH, SW22 SW_PUSH, SW23 SW_PUSH, SW24 SW_PUSH, SW25 SW_PUSH, SW26 SW_PUSH, SW27 SW_PUSH, SW28 SW_PUSH, SW29 SW_PUSH, SW3 SW_PUSH, SW30 SW_PUSH, SW31 SW_PUSH, SW32 SW_PUSH, SW33 SW_PUSH, SW34 SW_PUSH, SW35 SW_PUSH, SW36 SW_PUSH, SW37 SW_PUSH, SW38 SW_PUSH, SW39 SW_PUSH, SW4 SW_PUSH, SW40 SW_PUSH, SW41 SW_PUSH, SW42 SW_PUSH, SW5 SW_PUSH, SW6 SW_PUSH, SW7 SW_PUSH, SW8 SW_PUSH, SW9 SW_PUSH, U1 ProMicro, U2 ProMicro

Commit message: Change to CCDs
Parts:
- removed D23, D24, D25, D26, D27, D28, D29, D30, D31, D32, D33, D34, D35, D36, D37, D38, D39, D40, D41, D42: D, kbd:D3_TH_SMD_v2
- D1, D10, D11, D12, D13, D14, D15, D16, D17, D18, D19, D2, D20, D21, D22, D3, D4, D5, D6, D7, D8, D9: value D -> BAV70; footprint kbd:D3_TH_SMD_v2 -> Custom_Footprints:SOT-23_Annotated
- SW1, SW10, SW11, SW12, SW13, SW14, SW15, SW16, SW17, SW18, SW19, SW2, SW20, SW22, SW23, SW24, SW25, SW26, SW27, SW28, SW29, SW3, SW30, SW31, SW32, SW33, SW34, SW35, SW36, SW37, SW38, SW39, SW4, SW40, SW41, SW5, SW6, SW7, SW8, SW9: footprint kbd:keyswitch_cherrymx_alps_choc12_1u -> MX_Only:MXOnly-1U-NoLED
- SW21, SW42: footprint kbd:keyswitch_cherrymx_alps_choc12_1.5u -> MX_Only:MXOnly-1.5U-NoLED
- moved D22 216.2 mm to (69.9, -34.3)
- moved D20 147.1 mm to (83.5, -47.6)
- moved D21 143.6 mm to (79.0, -43.2)
- moved D19 137.7 mm to (74.4, -38.7)
- moved D16 122.7 mm to (83.5, -43.2)
- moved D13 122.0 mm to (74.4, -29.8)
- moved D15 118.1 mm to (79.0, -38.7)
- moved D17 117.6 mm to (74.4, -34.3)
- moved D18 115.6 mm to (69.9, -29.8)
- moved D14 115.3 mm to (69.9, -25.4)
- moved D8 105.2 mm to (79.0, -29.8)
- moved D11 101.2 mm to (83.5, -38.7)
- moved D12 98.9 mm to (79.0, -34.3)
- moved D10 95.0 mm to (83.5, -34.3)
- moved D7 94.5 mm to (69.9, -20.9)
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Connections:
- D1 pad 1: row0 -> Net-(D1-Pad1)
- D10 pad 1: row1 -> Net-(D10-Pad1)
- D11 pad 1: row1 -> Net-(D11-Pad1)
- D12 pad 1: row1 -> Net-(D12-Pad1)
- D13 pad 1: row2 -> Net-(D13-Pad1)
- D14 pad 1: row2 -> Net-(D14-Pad1)
- D15 pad 1: row2 -> Net-(D15-Pad1)
- D16 pad 1: row2 -> Net-(D16-Pad1)
- D17 pad 1: row2 -> Net-(D17-Pad1)
- D18 pad 1: row2 -> Net-(D18-Pad1)
- D19 pad 1: row3 -> Net-(D19-Pad1)
- D2 pad 1: row0 -> Net-(D2-Pad1)
- D20 pad 1: row3 -> Net-(D20-Pad1)
- D21 pad 1: row3 -> Net-(D21-Pad1)
- D22 pad 1: row0_r -> Net-(D22-Pad1)
- D3 pad 1: row0 -> Net-(D3-Pad1)
- D4 pad 1: row0 -> Net-(D4-Pad1)
- D5 pad 1: row0 -> Net-(D5-Pad1)
- D6 pad 1: row0 -> Net-(D6-Pad1)
- D7 pad 1: row1 -> Net-(D7-Pad1)
- D8 pad 1: row1 -> Net-(D8-Pad1)
- D9 pad 1: row1 -> Net-(D9-Pad1)
- SW1 pad 2: Net-(D1-Pad2) -> Net-(D1-Pad1)
- SW10 pad 2: Net-(D10-Pad2) -> Net-(D5-Pad2)
- SW11 pad 2: Net-(D11-Pad2) -> Net-(D6-Pad1)
- SW12 pad 2: Net-(D12-Pad2) -> Net-(D6-Pad2)
- SW13 pad 2: Net-(D13-Pad2) -> Net-(D7-Pad1)
- SW14 pad 2: Net-(D14-Pad2) -> Net-(D7-Pad2)
- SW15 pad 2: Net-(D15-Pad2) -> Net-(D8-Pad1)
- SW16 pad 2: Net-(D16-Pad2) -> Net-(D8-Pad2)
- SW17 pad 2: Net-(D17-Pad2) -> Net-(D9-Pad1)
- SW18 pad 2: Net-(D18-Pad2) -> Net-(D9-Pad2)
- SW19 pad 2: Net-(D19-Pad2) -> Net-(D10-Pad2)
- SW2 pad 2: Net-(D2-Pad2) -> Net-(D1-Pad2)
- SW20 pad 2: Net-(D20-Pad2) -> Net-(D11-Pad1)
- SW21 pad 2: Net-(D21-Pad2) -> Net-(D11-Pad2)
- SW22 pad 2: Net-(D22-Pad2) -> Net-(D12-Pad1)
- SW23 pad 2: Net-(D23-Pad2) -> Net-(D12-Pad2)
- SW24 pad 2: Net-(D24-Pad2) -> Net-(D13-Pad1)
- SW25 pad 2: Net-(D25-Pad2) -> Net-(D13-Pad2)
- SW26 pad 2: Net-(D26-Pad2) -> Net-(D14-Pad1)
- SW27 pad 2: Net-(D27-Pad2) -> Net-(D14-Pad2)
- SW28 pad 2: Net-(D28-Pad2) -> Net-(D15-Pad1)
- SW29 pad 2: Net-(D29-Pad2) -> Net-(D15-Pad2)
- SW3 pad 2: Net-(D3-Pad2) -> Net-(D2-Pad1)
- SW30 pad 2: Net-(D30-Pad2) -> Net-(D16-Pad1)
- SW31 pad 2: Net-(D31-Pad2) -> Net-(D16-Pad2)
- SW32 pad 2: Net-(D32-Pad2) -> Net-(D17-Pad1)
- SW33 pad 2: Net-(D33-Pad2) -> Net-(D17-Pad2)
- SW34 pad 2: Net-(D34-Pad2) -> Net-(D18-Pad1)
- SW35 pad 2: Net-(D35-Pad2) -> Net-(D18-Pad2)
- SW36 pad 2: Net-(D36-Pad2) -> Net-(D19-Pad1)
- SW37 pad 2: Net-(D37-Pad2) -> Net-(D19-Pad2)
- SW38 pad 2: Net-(D38-Pad2) -> Net-(D20-Pad1)
- SW39 pad 2: Net-(D39-Pad2) -> Net-(D20-Pad2)
- SW4 pad 2: Net-(D4-Pad2) -> Net-(D2-Pad2)
- SW40 pad 2: Net-(D40-Pad2) -> Net-(D21-Pad2)
- SW41 pad 2: Net-(D41-Pad2) -> Net-(D22-Pad1)
- SW42 pad 2: Net-(D42-Pad2) -> Net-(D22-Pad2)
- SW5 pad 2: Net-(D5-Pad2) -> Net-(D3-Pad1)
- SW6 pad 2: Net-(D6-Pad2) -> Net-(D3-Pad2)
- SW7 pad 2: Net-(D7-Pad2) -> Net-(D4-Pad1)
- SW8 pad 2: Net-(D8-Pad2) -> Net-(D4-Pad2)
- SW9 pad 2: Net-(D9-Pad2) -> Net-(D5-Pad1)
Routing:
- net col0_r: track 183.2 -> 0.00 mm, vias 1 -> 0
- net col0: track 182.3 -> 0.00 mm, vias 1 -> 0
- net row1: track 164.0 -> 0.00 mm
- net col1_r: track 161.3 -> 0.00 mm
- net col1: track 156.5 -> 0.00 mm, vias 1 -> 0
- net row2: track 153.9 -> 0.00 mm
- net col3_r: track 148.5 -> 0.00 mm, vias 1 -> 0
- net row0: track 142.3 -> 0.00 mm
- net col3: track 141.3 -> 0.00 mm, vias 1 -> 0
- net col2_r: track 141.1 -> 0.00 mm, vias 1 -> 0
- net row2_r: track 137.6 -> 0.00 mm, vias 2 -> 0
- net col2: track 135.2 -> 0.00 mm, vias 1 -> 0
- net row1_r: track 134.3 -> 0.00 mm
- net col4_r: track 129.6 -> 0.00 mm, vias 1 -> 0
- net row0_r: track 127.8 -> 0.00 mm
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Other:
- outline, holes or cut-outs redrawn
- board text removed: "Corne Light v2.0 PCB Designed by foostan"

Commit message: Place CCDs
Parts:
- moved D18 229.9 mm to (269.2, 84.8), turned to 270 degrees
- moved D15 217.0 mm to (269.2, 65.7), turned to 270 degrees
- moved D12 206.7 mm to (269.2, 46.7), turned to 270 degrees
- moved D19 195.7 mm to (231.2, 78.4), turned to 270 degrees
- moved D21 189.1 mm to (202.7, 99.8), turned to 270 degrees
- moved D16 180.2 mm to (231.2, 60.2), turned to 270 degrees
- moved D22 178.4 mm to (180.9, 105.4), turned to 300 degrees
- moved D13 172.4 mm to (231.2, 41.9), turned to 270 degrees
- moved D20 170.1 mm to (193.2, 82.4), turned to 270 degrees
- moved D17 153.7 mm to (193.2, 63.3), turned to 270 degrees
- moved D11 148.4 mm to (119.0, 105.4), turned to 240 degrees
- moved D14 141.6 mm to (193.2, 44.3), turned to 270 degrees
- moved D10 134.9 mm to (98.2, 99.8), turned to 270 degrees
- moved D9 112.8 mm to (107.7, 82.4), turned to 270 degrees
- moved D7 112.3 mm to (31.7, 84.8), turned to 270 degrees
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Connections:
- SW19 pad 2: Net-(D10-Pad2) -> Net-(D10-Pad1)
- SW22 pad 2: Net-(D12-Pad1) -> Net-(D12-Pad2)
- SW23 pad 2: Net-(D12-Pad2) -> Net-(D12-Pad1)
- SW24 pad 2: Net-(D13-Pad1) -> Net-(D13-Pad2)
- SW25 pad 2: Net-(D13-Pad2) -> Net-(D13-Pad1)
- SW26 pad 2: Net-(D14-Pad1) -> Net-(D14-Pad2)
- SW27 pad 2: Net-(D14-Pad2) -> Net-(D14-Pad1)
- SW28 pad 2: Net-(D15-Pad1) -> Net-(D15-Pad2)
- SW29 pad 2: Net-(D15-Pad2) -> Net-(D15-Pad1)
- SW30 pad 2: Net-(D16-Pad1) -> Net-(D16-Pad2)
- SW31 pad 2: Net-(D16-Pad2) -> Net-(D16-Pad1)
- SW32 pad 2: Net-(D17-Pad1) -> Net-(D17-Pad2)
- SW33 pad 2: Net-(D17-Pad2) -> Net-(D17-Pad1)
- SW34 pad 2: Net-(D18-Pad1) -> Net-(D18-Pad2)
- SW35 pad 2: Net-(D18-Pad2) -> Net-(D18-Pad1)
- SW36 pad 2: Net-(D19-Pad1) -> Net-(D19-Pad2)
- SW37 pad 2: Net-(D19-Pad2) -> Net-(D19-Pad1)
- SW38 pad 2: Net-(D20-Pad1) -> Net-(D20-Pad2)
- SW39 pad 2: Net-(D20-Pad2) -> Net-(D20-Pad1)
- SW41 pad 2: Net-(D22-Pad1) -> Net-(D22-Pad2)
- SW42 pad 2: Net-(D22-Pad2) -> Net-(D22-Pad1)

Commit message: Route mcu
Connections:
- SW21 pad 1: col5 -> Net-(D11-Pad2)
- SW21 pad 2: Net-(D11-Pad2) -> col5
- SW41 pad 1: col4_r -> Net-(D22-Pad2)
- SW41 pad 2: Net-(D22-Pad2) -> col4_r
Routing:
- net row2_r: track 0.00 -> 80.0 mm
- net row1_r: track 0.00 -> 79.5 mm
- net row2: track 0.00 -> 79.3 mm
- net row0_r: track 0.00 -> 78.9 mm
- net row1: track 0.00 -> 78.7 mm
- net row0: track 0.00 -> 78.7 mm
- net col5: track 0.00 -> 65.9 mm
- net col4: track 0.00 -> 64.6 mm
- net col5_r: track 0.00 -> 64.1 mm
- net col3_r: track 0.00 -> 63.9 mm
- net col3: track 0.00 -> 63.9 mm
- net col4_r: track 0.00 -> 60.1 mm
- net col2_r: track 0.00 -> 38.0 mm
- net col1_r: track 0.00 -> 38.0 mm
- net col0_r: track 0.00 -> 38.0 mm
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
Commit message: Curve cols
Routing:
- net col4_r: track 60.1 -> 59.5 mm
- net col5_r: track 64.1 -> 63.6 mm
- net col3_r: track 63.9 -> 63.4 mm
- net col5: track 65.9 -> 65.4 mm
- net col3: track 63.9 -> 63.4 mm
- net col4: track 64.6 -> 64.0 mm

Commit message: Route matrix and others
Routing:
- net col0_r: track 38.0 -> 191.2 mm, vias 0 -> 1
- net col0: track 38.0 -> 162.0 mm, vias 0 -> 1
- net col1_r: track 38.0 -> 156.5 mm, vias 0 -> 1
- net col1: track 38.0 -> 140.9 mm, vias 0 -> 1
- net col2_r: track 38.0 -> 135.5 mm, vias 0 -> 1
- net reset_r: track 0.00 -> 88.4 mm
- net col2: track 38.0 -> 119.8 mm, vias 0 -> 1
- net data: track 0.00 -> 79.1 mm
- net col3_r: track 63.4 -> 138.8 mm, vias 0 -> 1
- net GNDA: track 0.00 -> 75.0 mm
- net GND: track 0.00 -> 65.6 mm
- net data_r: track 0.00 -> 62.5 mm
- net reset: track 0.00 -> 62.4 mm
- net col3: track 63.4 -> 123.3 mm, vias 0 -> 1
- net col4_r: track 59.5 -> 113.7 mm, vias 0 -> 1
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
Commit message: Add new text
Parts:
- added REF**: 1.62mm, TestPoint:1.62, F.Cu at (278.7, 119.8)
- added REF**: 1.6mm, TestPoint:1.6mm, F.Cu at (278.7, 111.2)
- added REF**: 1.59mm, TestPoint:1.59mm, F.Cu at (278.7, 106.8)
- added REF**: 1.58mm, TestPoint:1.58mm, F.Cu at (278.7, 102.4)
- added REF**: 1.61mm, TestPoint:1.61, F.Cu at (278.7, 115.6)
Routing:
- added copper zone on B.Cu, net (none)
- added copper zone on F.Cu, net (none)
Other:
- board text added: "Edited by Swiftrax"
Changed lines of the file:
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@@
   (general
     (thickness 1.6)
-    (drawings 739)
+    (drawings 743)
     (tracks 3247)
     (zones 0)
-    (modules 102)
+    (modules 107)
     (nets 91)
   )
@@
   )
   (setup
-    (last_trace_width 0.35)
+    (last_trace_width 0.25)
     (user_trace_width 0.2032)
     (user_trace_width 0.254)
@@
     (mod_text_size 1 1)
     (mod_text_width 0.15)
-    (pad_size 0.8128 0.8128)
-    (pad_drill 0.8128)
+    (pad_size 5 1.61)
+    (pad_drill 5)
     (pad_to_mask_clearance 0.2)
     (aux_axis_origin 74.8395 91.6855)
@@
     (diff_pair_gap 0.00001)
   )
+  (module TestPoint:1.62 (layer F.Cu)
+    (at 278.7125 119.845)
+    (fp_text reference REF** (at 0 1.9) (layer F.Fab)
+      (effects (font (size 1 1) (thickness 0.15)))
+    )
+    (fp_text value 1.62mm (at 0 -1.9) (layer F.SilkS)
+      (effects (font (size 1 1) (thickness 0.15)))
+    )
+    (pad 1 thru_hole oval (at 0 0) (size 5 1.62) (drill oval 5 1.62) (layers *.Cu *.Mask))
+  )
+  (module TestPoint:1.6mm (layer F.Cu)
+    (at 278.7125 111.245)
+    (fp_text reference REF** (at 0 1.9) (layer F.Fab)
+      (effects (font (size 1 1) (thickness 0.15)))
+    )
+    (fp_text value 1.6mm (at 0 -1.9) (layer F.SilkS)
+      (effects (font (size 1 1) (thickness 0.15)))
+    )
+    (pad 1 thru_hole oval (at 0 0) (size 5 1.6) (drill oval 5 1.6) (layers *.Cu *.Mask))
+  )
+  (module TestPoint:1.59mm (layer F.Cu)
+    (at 278.7125 106.845)
+    (fp_text reference REF** (at 0 1.9) (layer F.Fab)
+      (effects (font (size 1 1) (thickness 0.15)))
+    )
+    (fp_text value 1.59mm (at 0 -1.9) (layer F.SilkS)
+      (effects (font (size 1 1) (thickness 0.15)))
+    )
+    (pad 1 thru_hole oval (at 0 0) (size 5 1.59) (drill oval 5 1.59) (layers *.Cu *.Mask))
+  )
+  (module TestPoint:1.58mm (layer F.Cu)
+    (at 278.7125 102.445)
+    (fp_text reference REF** (at 0 1.9) (layer F.Fab)
+      (effects (font (size 1 1) (thickness 0.15)))
+    )
+    (fp_text value 1.58mm (at 0 -1.9) (layer F.SilkS)
+      (effects (font (size 1 1) (thickness 0.15)))
+    )
+    (pad 1 thru_hole oval (at 0 0) (size 5 1.58) (drill oval 5 1.58) (layers *.Cu *.Mask))
+  )
+  (module TestPoint:1.61 (layer F.Cu)
+    (at 278.7125 115.645)
+    (fp_text reference REF** (at 0 1.9) (layer F.Fab)
+      (effects (font (size 1 1) (thickness 0.15)))
+    )
+    (fp_text value 1.61mm (at 0 -1.9) (layer F.SilkS)
+      (effects (font (size 1 1) (thickness 0.15)))
+    )
+    (pad 1 thru_hole oval (at 0 0) (size 5 1.61) (drill oval 5 1.61) (layers *.Cu *.Mask))
+  )
   (module Custom_Footprints:SOT-23_Annotated (layer B.Cu)
     (at 180.928927 105.400762 300)
@@
     )
   )
+  (gr_text "Edited by Swiftrax" (at 46.7125 70.945) (layer B.Mask)
+    (effects (font (size 1.5 1.5) (thickness 0.31)) (justify mirror))
+  )
+  (gr_text "Edited by Swiftrax" (at 46.7125 70.945) (layer B.Cu)
+    (effects (font (size 1.5 1.5) (thickness 0.3)) (justify mirror))
+  )
+  (gr_text "Edited by Swiftrax" (at 248.7125 70.445) (layer B.Mask)
+    (effects (font (size 1.5 1.5) (thickness 0.31)) (justify mirror))
+  )
+  (gr_text "Edited by Swiftrax" (at 248.7125 70.445) (layer B.Cu)
+    (effects (font (size 1.5 1.5) (thickness 0.3)) (justify mirror))
+  )
   (gr_line (start 50.575196 36.92899) (end 13.688928 36.928989) (layer Edge.Cuts) (width 0.2))
   (gr_line (start 19.848845 93.652214) (end 19.780265 93.873192) (layer Edge.Cuts) (width 0.2))
@@
   (segment (start 174.650771 105.009736) (end 174.595684 104.95465) (width 0.5) (layer B.Cu) (net 90))
   (segment (start 179.606203 105.009736) (end 174.650771 105.009736) (width 0.5) (layer B.Cu) (net 90))
+  (zone (net 0) (net_name "") (layer F.Cu) (hatch edge 0.508)
+    (connect_pads (clearance 0.508))
+    (min_thickness 0.254)
+    (fill yes (arc_segments 32) (thermal_gap 0.508) (thermal_bridge_width 0.508))
+    (polygon
+      (pts
+        (xy 237.5125 27.245) (xy 237.5125 31.245) (xy 243.9125 31.245) (xy 243.9125 27.245)
+      )
+    )
+  )
+  (zone (net 0) (net_name "") (layer B.Cu) (hatch edge 0.508)
+    (connect_pads (clearance 0.508))
+    (min_thickness 0.254)
+    (fill yes (arc_segments 32) (thermal_gap 0.508) (thermal_bridge_width 0.508))
+    (polygon
+      (pts
+        (xy 237.5125 27.245) (xy 237.5125 31.245) (xy 243.9125 31.245) (xy 243.9125 27.245)
+      )
+    )
+  )
+  (zone (net 0) (net_name "") (layer F.Cu) (hatch edge 0.508)
+    (connect_pads (clearance 0.508))
+    (min_thickness 0.254)
+    (fill yes (arc_segments 32) (thermal_gap 0.508) (thermal_bridge_width 0.508))
+    (polygon
+      (pts
+        (xy 56.9125 27.445) (xy 56.9125 31.445) (xy 63.3125 31.445) (xy 63.3125 27.445)
+      )
+    )
+  )
+  (zone (net 0) (net_name "") (layer B.Cu) (hatch edge 0.508)
+    (connect_pads (clearance 0.508))
+    (min_thickness 0.254)
+    (fill yes (arc_segments 32) (thermal_gap 0.508) (thermal_bridge_width 0.508))
+    (polygon
+      (pts
+        (xy 56.9125 27.445) (xy 56.9125 31.445) (xy 63.3125 31.445) (xy 63.3125 27.445)
+      )
+    )
+  )
+  (zone (net 0) (net_name "") (layer F.Cu) (hatch edge 0.508)
+    (connect_pads (clearance 0.508))
+    (min_thickness 0.254)
+    (fill yes (arc_segments 32) (thermal_gap 0.508) (thermal_bridge_width 0.508))
+    (polygon
+      (pts
+        (xy 94.9125 27.445) (xy 94.9125 31.445) (xy 101.3125 31.445) (xy 101.3125 27.445)
+      )
+    )
+  )
+  (zone (net 0) (net_name "") (layer B.Cu) (hatch edge 0.508)
+    (connect_pads (clearance 0.508))
+    (min_thickness 0.254)
+    (fill yes (arc_segments 32) (thermal_gap 0.508) (thermal_bridge_width 0.508))
+    (polygon
+      (pts
+        (xy 199.5125 27.245) (xy 199.5125 31.245) (xy 205.9125 31.245) (xy 205.9125 27.245)
+      )
+    )
+  )
 )

Commit message: Make Gerbers
Parts:
- added G***: LOGO, kbd:Corne_Art, B.Cu at (150.2, 73.4)

Commit message: Change Art
Parts:
- removed the G*** at (150.2, 73.4)
- added G***: LOGO, kbd:CapyBara_900, B.Cu at (177.0, 89.6)
- added G***: LOGO, kbd:CapyBara_900, B.Cu at (123.3, 89.4)
